File: PCB_Design/bldc_pcb_design/bldc_pcb_design.sch (KiCad schematic (older format))
At the start: 74 parts, among them IC1 DRV8305NPHPR, J1 Conn_01x06_Female, SW1 BOOT, SW2 RESET, U1 ESP32-WROOM-32D, U10 DS18S20Z+, U2 AS5600-ASOT, U3 LM2672M-3.3, U4 CSD18532NQ5BT, U5 CSD18532NQ5BT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

Commit message: Re-routed DRV8305 using corrected underneath GND pad footprint, back mounted Temp sensor
Parts:
- added R16, R17: 10k, Resistor_SMD:R_0603_1608Metric, symbol Device:R
- added T1, T2: BC847, BC847:BC847, symbol BC847:BC847
- IC1: footprint DRV8305NPHPR:DRV8305NPHPR -> DRV8305NPHPR:DRV8305NEPHPRQ1_with_GND_pads
Connections:
- net BOOT: now also T2.2
- net CTS: no longer J1.5 (Pin_5)
- net DTR: no longer J1.1 (Pin_1)
- net RESET: now also T1.3
- new net: R16.1, T1.1
- new net: R17.2, T2.1
- new net ~DTR: J1.1 (Pin_1), R16.2, T2.3
- new net ~RTS: J1.5 (Pin_5), R17.1, T1.2
Other:
- note added: "MCU Auto Reset Circuitry"
- note added: "Power Connector\n Pads\n"
- note removed: "Power Connector Pads\n"
- moved on the sheet: C1, C12, C13, C14, C15, C18, C8, C9, H1, H2, H5, H8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
